Commit message: using figer tool

File: force_sensor/urdf/grabber.xacro (robot description, xacro)
@@ -27,5 +27,5 @@
         <origin xyz="0 0 0" rpy="0 0 0"/>
         <geometry>
-          <mesh filename="package://force_sensor/meshes/collision/grabber.stl"/>
+          <mesh filename="package://force_sensor/meshes/collision/finger_tool.stl"/>
         </geometry>
         <material name="White"/>
@@ -73,5 +73,5 @@
         <origin xyz="0 0 0" rpy="0 0 0"/>
         <geometry>
-          <mesh filename="package://force_sensor/meshes/visual/grabber.stl"/>
+          <mesh filename="package://force_sensor/meshes/visual/finger_tool.stl"/>
         </geometry>
         <material name="White"/>

Commit message: the tool offset is work

File: force_sensor/urdf/grabber.xacro (robot description, xacro)
@@ -78,5 +78,5 @@
       </visual>
       <inertial>
-        <mass value="1e-5" />
+        <mass value="2.0" />
         <origin xyz="0 0 0" rpy="0 0 0"/>
         <inertia ixx="1e-6" ixy="0" ixz="0" iyy="1e-6" iyz="0" izz="1e-6" />
